Commit message: Slerp bug

File: urdf/robot_model.urdf (robot description, URDF)
Before this commit: robot continuum_robot, 41 links, 40 joints
Links:
- removed link S1L0
- removed link S1L1
- removed link S1L10
- removed link S1L11
- removed link S1L12
- removed link S1L13
- removed link S1L14
- removed link S1L15
- removed link S1L16
- removed link S1L17
- removed link S1L18
- removed link S1L19
- removed link S1L2
- removed link S1L3
- removed link S1L4
- removed link S1L5
- removed link S1L6
- removed link S1L7
- removed link S1L8
- removed link S1L9
- removed link S2L0
- removed link S2L1
- removed link S2L2
- removed link S2L3
- removed link S2L4
- removed link S2L5
- removed link S2L6
- removed link S2L7
- removed link S2L8
- removed link S2L9
- link S0L0: geometry visual cylinder length=0.1 radius=0.4
- link S0L1: geometry visual cylinder length=0.1 radius=0.4
- link S0L2: geometry visual cylinder length=0.1 radius=0.4
- link S0L3: geometry visual cylinder length=0.1 radius=0.4
- link S0L4: geometry visual cylinder length=0.1 radius=0.4
- link S0L5: geometry visual cylinder length=0.1 radius=0.4
- link S0L6: geometry visual cylinder length=0.1 radius=0.4
- link S0L7: geometry visual cylinder length=0.1 radius=0.4
- link S0L8: geometry visual cylinder length=0.1 radius=0.4
- link S0L9: geometry visual cylinder length=0.1 radius=0.4
Joints:
- removed joint S1J0
- removed joint S1J1
- removed joint S1J10
- removed joint S1J11
- removed joint S1J12
- removed joint S1J13
- removed joint S1J14
- removed joint S1J15
- removed joint S1J16
- removed joint S1J17
- removed joint S1J18
- removed joint S1J19
- removed joint S1J2
- removed joint S1J3
- removed joint S1J4
- removed joint S1J5
- removed joint S1J6
- removed joint S1J7
- removed joint S1J8
- removed joint S1J9
- removed joint S2J0
- removed joint S2J1
- removed joint S2J2
- removed joint S2J3
- removed joint S2J4
- removed joint S2J5
- removed joint S2J6
- removed joint S2J7
- removed joint S2J8
- removed joint S2J9

Commit message: Solve segments issu

File: urdf/robot_model.urdf (robot description, URDF)
Before this commit: robot continuum_robot, 11 links, 10 joints
Links:
- added link S1L0; visual cylinder length=0.1 radius=0.3
- added link S1L1; visual cylinder length=0.1 radius=0.3
- added link S1L10; visual cylinder length=0.1 radius=0.3
- added link S1L11; visual cylinder length=0.1 radius=0.3
- added link S1L12; visual cylinder length=0.1 radius=0.3
- added link S1L13; visual cylinder length=0.1 radius=0.3
- added link S1L14; visual cylinder length=0.1 radius=0.3
- added link S1L15; visual cylinder length=0.1 radius=0.3
- added link S1L16; visual cylinder length=0.1 radius=0.3
- added link S1L17; visual cylinder length=0.1 radius=0.3
- added link S1L18; visual cylinder length=0.1 radius=0.3
- added link S1L19; visual cylinder length=0.1 radius=0.3
- added link S1L2; visual cylinder length=0.1 radius=0.3
- added link S1L3; visual cylinder length=0.1 radius=0.3
- added link S1L4; visual cylinder length=0.1 radius=0.3
- added link S1L5; visual cylinder length=0.1 radius=0.3
- added link S1L6; visual cylinder length=0.1 radius=0.3
- added link S1L7; visual cylinder length=0.1 radius=0.3
- added link S1L8; visual cylinder length=0.1 radius=0.3
- added link S1L9; visual cylinder length=0.1 radius=0.3
- added link S2L0; visual cylinder length=0.1 radius=0.2
- added link S2L1; visual cylinder length=0.1 radius=0.2
- added link S2L2; visual cylinder length=0.1 radius=0.2
- added link S2L3; visual cylinder length=0.1 radius=0.2
- added link S2L4; visual cylinder length=0.1 radius=0.2
- added link S2L5; visual cylinder length=0.1 radius=0.2
- added link S2L6; visual cylinder length=0.1 radius=0.2
- added link S2L7; visual cylinder length=0.1 radius=0.2
- added link S2L8; visual cylinder length=0.1 radius=0.2
- added link S2L9; visual cylinder length=0.1 radius=0.2
- link S0L0: geometry visual box size=1 1 0.5
Joints:
- added joint S1J0: type floating, parent base_link, child S1L0
- added joint S1J1: type floating, parent base_link, child S1L1
- added joint S1J10: type floating, parent base_link, child S1L10
- added joint S1J11: type floating, parent base_link, child S1L11
- added joint S1J12: type floating, parent base_link, child S1L12
- added joint S1J13: type floating, parent base_link, child S1L13
- added joint S1J14: type floating, parent base_link, child S1L14
- added joint S1J15: type floating, parent base_link, child S1L15
- added joint S1J16: type floating, parent base_link, child S1L16
- added joint S1J17: type floating, parent base_link, child S1L17
- added joint S1J18: type floating, parent base_link, child S1L18
- added joint S1J19: type floating, parent base_link, child S1L19
- added joint S1J2: type floating, parent base_link, child S1L2
- added joint S1J3: type floating, parent base_link, child S1L3
- added joint S1J4: type floating, parent base_link, child S1L4
- added joint S1J5: type floating, parent base_link, child S1L5
- added joint S1J6: type floating, parent base_link, child S1L6
- added joint S1J7: type floating, parent base_link, child S1L7
- added joint S1J8: type floating, parent base_link, child S1L8
- added joint S1J9: type floating, parent base_link, child S1L9
- added joint S2J0: type floating, parent base_link, child S2L0
- added joint S2J1: type floating, parent base_link, child S2L1
- added joint S2J2: type floating, parent base_link, child S2L2
- added joint S2J3: type floating, parent base_link, child S2L3
- added joint S2J4: type floating, parent base_link, child S2L4
- added joint S2J5: type floating, parent base_link, child S2L5
- added joint S2J6: type floating, parent base_link, child S2L6
- added joint S2J7: type floating, parent base_link, child S2L7
- added joint S2J8: type floating, parent base_link, child S2L8
- added joint S2J9: type floating, parent base_link, child S2L9

Commit message: snake

File: urdf/robot_model.urdf (robot description, URDF)
Before this commit: robot continuum_robot, 41 links, 40 joints
Links:
- removed link S1L0
- removed link S1L1
- removed link S1L10
- removed link S1L11
- removed link S1L12
- removed link S1L13
- removed link S1L14
- removed link S1L15
- removed link S1L16
- removed link S1L17
- removed link S1L18
- removed link S1L19
- removed link S1L2
- removed link S1L3
- removed link S1L4
- removed link S1L5
- removed link S1L6
- removed link S1L7
- removed link S1L8
- removed link S1L9
- removed link S2L0
- removed link S2L1
- removed link S2L2
- removed link S2L3
- removed link S2L4
- removed link S2L5
- removed link S2L6
- removed link S2L7
- removed link S2L8
- removed link S2L9
- added link S0L10; visual cylinder length=0.1 radius=0.4
- added link S0L11; visual cylinder length=0.1 radius=0.4
- added link S0L12; visual cylinder length=0.1 radius=0.4
- added link S0L13; visual cylinder length=0.1 radius=0.4
- added link S0L14; visual cylinder length=0.1 radius=0.4
- added link S0L15; visual cylinder length=0.1 radius=0.4
- added link S0L16; visual cylinder length=0.1 radius=0.4
- added link S0L17; visual cylinder length=0.1 radius=0.4
- added link S0L18; visual cylinder length=0.1 radius=0.4
- added link S0L19; visual cylinder length=0.1 radius=0.4
Joints:
- removed joint S1J0
- removed joint S1J1
- removed joint S1J10
- removed joint S1J11
- removed joint S1J12
- removed joint S1J13
- removed joint S1J14
- removed joint S1J15
- removed joint S1J16
- removed joint S1J17
- removed joint S1J18
- removed joint S1J19
- removed joint S1J2
- removed joint S1J3
- removed joint S1J4
- removed joint S1J5
- removed joint S1J6
- removed joint S1J7
- removed joint S1J8
- removed joint S1J9
- removed joint S2J0
- removed joint S2J1
- removed joint S2J2
- removed joint S2J3
- removed joint S2J4
- removed joint S2J5
- removed joint S2J6
- removed joint S2J7
- removed joint S2J8
- removed joint S2J9
- added joint S0J10: type floating, parent base_link, child S0L10
- added joint S0J11: type floating, parent base_link, child S0L11
- added joint S0J12: type floating, parent base_link, child S0L12
- added joint S0J13: type floating, parent base_link, child S0L13
- added joint S0J14: type floating, parent base_link, child S0L14
- added joint S0J15: type floating, parent base_link, child S0L15
- added joint S0J16: type floating, parent base_link, child S0L16
- added joint S0J17: type floating, parent base_link, child S0L17
- added joint S0J18: type floating, parent base_link, child S0L18
- added joint S0J19: type floating, parent base_link, child S0L19

Commit message: final

File: urdf/robot_model.urdf (robot description, URDF)
Before this commit: robot continuum_robot, 21 links, 20 joints
Links:
- removed link S0L10
- removed link S0L11
- removed link S0L12
- removed link S0L13
- removed link S0L14
- removed link S0L15
- removed link S0L16
- removed link S0L17
- removed link S0L18
- removed link S0L19
- removed link S0L6
- removed link S0L7
- removed link S0L8
- removed link S0L9
- added link S1L0; visual cylinder length=0.1 radius=0.3
- added link S1L1; visual cylinder length=0.1 radius=0.3
- added link S1L2; visual cylinder length=0.1 radius=0.3
- added link S1L3; visual cylinder length=0.1 radius=0.3
- added link S1L4; visual cylinder length=0.1 radius=0.3
- added link S1L5; visual cylinder length=0.1 radius=0.3
Joints:
- removed joint S0J10
- removed joint S0J11
- removed joint S0J12
- removed joint S0J13
- removed joint S0J14
- removed joint S0J15
- removed joint S0J16
- removed joint S0J17
- removed joint S0J18
- removed joint S0J19
- removed joint S0J6
- removed joint S0J7
- removed joint S0J8
- removed joint S0J9
- added joint S1J0: type floating, parent base_link, child S1L0
- added joint S1J1: type floating, parent base_link, child S1L1
- added joint S1J2: type floating, parent base_link, child S1L2
- added joint S1J3: type floating, parent base_link, child S1L3
- added joint S1J4: type floating, parent base_link, child S1L4
- added joint S1J5: type floating, parent base_link, child S1L5

Commit message: Final update

File: urdf/robot_model.urdf (robot description, URDF)
Before this commit: robot continuum_robot, 13 links, 12 joints
Links:
- added link S0L10; visual cylinder length=0.1 radius=0.3
- added link S0L11; visual cylinder length=0.1 radius=0.3
- added link S0L12; visual cylinder length=0.1 radius=0.3
- added link S0L13; visual cylinder length=0.1 radius=0.3
- added link S0L14; visual cylinder length=0.1 radius=0.3
- added link S0L15; visual cylinder length=0.1 radius=0.3
- added link S0L16; visual cylinder length=0.1 radius=0.3
- added link S0L17; visual cylinder length=0.1 radius=0.3
- added link S0L18; visual cylinder length=0.1 radius=0.3
- added link S0L19; visual cylinder length=0.1 radius=0.3
- added link S0L20; visual cylinder length=0.1 radius=0.3
- added link S0L21; visual cylinder length=0.1 radius=0.3
- added link S0L22; visual cylinder length=0.1 radius=0.3
- added link S0L23; visual cylinder length=0.1 radius=0.3
- added link S0L24; visual cylinder length=0.1 radius=0.3
- added link S0L25; visual cylinder length=0.1 radius=0.3
- added link S0L26; visual cylinder length=0.1 radius=0.3
- added link S0L27; visual cylinder length=0.1 radius=0.3
- added link S0L28; visual cylinder length=0.1 radius=0.3
- added link S0L29; visual cylinder length=0.1 radius=0.3
- added link S0L6; visual cylinder length=0.1 radius=0.3
- added link S0L7; visual cylinder length=0.1 radius=0.3
- added link S0L8; visual cylinder length=0.1 radius=0.3
- added link S0L9; visual cylinder length=0.1 radius=0.3
- added link S1L10; visual cylinder length=0.1 radius=0.3
- added link S1L11; visual cylinder length=0.1 radius=0.3
- added link S1L12; visual cylinder length=0.1 radius=0.3
- added link S1L13; visual cylinder length=0.1 radius=0.3
- added link S1L14; visual cylinder length=0.1 radius=0.3
- added link S1L15; visual cylinder length=0.1 radius=0.3
- added link S1L16; visual cylinder length=0.1 radius=0.3
- added link S1L17; visual cylinder length=0.1 radius=0.3
- added link S1L18; visual cylinder length=0.1 radius=0.3
- added link S1L19; visual cylinder length=0.1 radius=0.3
- added link S1L20; visual cylinder length=0.1 radius=0.3
- added link S1L21; visual cylinder length=0.1 radius=0.3
- added link S1L22; visual cylinder length=0.1 radius=0.3
- added link S1L23; visual cylinder length=0.1 radius=0.3
- added link S1L24; visual cylinder length=0.1 radius=0.3
- added link S1L25; visual cylinder length=0.1 radius=0.3
- added link S1L26; visual cylinder length=0.1 radius=0.3
- added link S1L27; visual cylinder length=0.1 radius=0.3
- added link S1L28; visual cylinder length=0.1 radius=0.3
- added link S1L29; visual cylinder length=0.1 radius=0.3
- added link S1L6; visual cylinder length=0.1 radius=0.3
- added link S1L7; visual cylinder length=0.1 radius=0.3
- added link S1L8; visual cylinder length=0.1 radius=0.3
- added link S1L9; visual cylinder length=0.1 radius=0.3
- added link S2L0; visual cylinder length=0.1 radius=0.2
- added link S2L1; visual cylinder length=0.1 radius=0.2
- added link S2L2; visual cylinder length=0.1 radius=0.2
- added link S2L3; visual cylinder length=0.1 radius=0.2
- added link S2L4; visual cylinder length=0.1 radius=0.2
- added link S2L5; visual cylinder length=0.1 radius=0.2
- link S0L1: geometry visual cylinder length=0.1 radius=0.3
- link S0L2: geometry visual cylinder length=0.1 radius=0.3
- link S0L3: geometry visual cylinder length=0.1 radius=0.3
- link S0L4: geometry visual cylinder length=0.1 radius=0.3
- link S0L5: geometry visual cylinder length=0.1 radius=0.3
Joints:
- added joint S0J10: type floating, parent base_link, child S0L10
- added joint S0J11: type floating, parent base_link, child S0L11
- added joint S0J12: type floating, parent base_link, child S0L12
- added joint S0J13: type floating, parent base_link, child S0L13
- added joint S0J14: type floating, parent base_link, child S0L14
- added joint S0J15: type floating, parent base_link, child S0L15
- added joint S0J16: type floating, parent base_link, child S0L16
- added joint S0J17: type floating, parent base_link, child S0L17
- added joint S0J18: type floating, parent base_link, child S0L18
- added joint S0J19: type floating, parent base_link, child S0L19
- added joint S0J20: type floating, parent base_link, child S0L20
- added joint S0J21: type floating, parent base_link, child S0L21
- added joint S0J22: type floating, parent base_link, child S0L22
- added joint S0J23: type floating, parent base_link, child S0L23
- added joint S0J24: type floating, parent base_link, child S0L24
- added joint S0J25: type floating, parent base_link, child S0L25
- added joint S0J26: type floating, parent base_link, child S0L26
- added joint S0J27: type floating, parent base_link, child S0L27
- added joint S0J28: type floating, parent base_link, child S0L28
- added joint S0J29: type floating, parent base_link, child S0L29
- added joint S0J6: type floating, parent base_link, child S0L6
- added joint S0J7: type floating, parent base_link, child S0L7
- added joint S0J8: type floating, parent base_link, child S0L8
- added joint S0J9: type floating, parent base_link, child S0L9
- added joint S1J10: type floating, parent base_link, child S1L10
- added joint S1J11: type floating, parent base_link, child S1L11
- added joint S1J12: type floating, parent base_link, child S1L12
- added joint S1J13: type floating, parent base_link, child S1L13
- added joint S1J14: type floating, parent base_link, child S1L14
- added joint S1J15: type floating, parent base_link, child S1L15
- added joint S1J16: type floating, parent base_link, child S1L16
- added joint S1J17: type floating, parent base_link, child S1L17
- added joint S1J18: type floating, parent base_link, child S1L18
- added joint S1J19: type floating, parent base_link, child S1L19
- added joint S1J20: type floating, parent base_link, child S1L20
- added joint S1J21: type floating, parent base_link, child S1L21
- added joint S1J22: type floating, parent base_link, child S1L22
- added joint S1J23: type floating, parent base_link, child S1L23
- added joint S1J24: type floating, parent base_link, child S1L24
- added joint S1J25: type floating, parent base_link, child S1L25
- added joint S1J26: type floating, parent base_link, child S1L26
- added joint S1J27: type floating, parent base_link, child S1L27
- added joint S1J28: type floating, parent base_link, child S1L28
- added joint S1J29: type floating, parent base_link, child S1L29
- added joint S1J6: type floating, parent base_link, child S1L6
- added joint S1J7: type floating, parent base_link, child S1L7
- added joint S1J8: type floating, parent base_link, child S1L8
- added joint S1J9: type floating, parent base_link, child S1L9
- added joint S2J0: type floating, parent base_link, child S2L0
- added joint S2J1: type floating, parent base_link, child S2L1
- added joint S2J2: type floating, parent base_link, child S2L2
- added joint S2J3: type floating, parent base_link, child S2L3
- added joint S2J4: type floating, parent base_link, child S2L4
- added joint S2J5: type floating, parent base_link, child S2L5
